File: lampe.brd (EAGLE design)
At the start: 86.2 x 21 mm, 29 parts, among them T3 LTR-4206, X1 USBPCB

Commit message: feat(lampe): Fix silk screen and some values
Parts:
- removed R13: 1k8, rcl:0207/7
- added R12: 68k, rcl:0207/7
- R1: value 100 -> 1k8
- R5: value 68k -> 100
- moved R1 38.1 mm to (9.00, 10.5), turned to 180 degrees
- moved R5 33.9 mm to (52.5, 15.5), turned to 270 degrees
- moved R4 10.4 mm to (49.8, 15.5)
- moved R6 9.90 mm to (52.5, 5.50), turned to 270 degrees
- moved R2 7.63 mm to (44.0, 10.5), turned to 90 degrees
- moved R3 5.77 mm to (46.8, 15.5)
Connections:
- net +5V: now also R12.1; no longer R5.1
- net LED1: now also R2.2; no longer R6.2
- net LED2: now also R3.2; no longer R1.2
- net LED3: now also R4.2; no longer R2.2
- net LED4: now also R5.2; no longer R3.2
- net LIGHT: now also R12.2; no longer R5.2
- net N$1: now also R3.1; no longer R1.1
- net N$10: now also R5.1; no longer R3.1
- net N$17: now also R2.1; no longer R6.1
- net N$2: now also R6.2; no longer R4.2
- net N$29: now also R1.2; no longer R13.2
- net N$3: now also R4.1; no longer R2.1
- net PIEZO: now also R1.1; no longer R13.1
- net R1: now also R6.1; no longer R4.1
